File: LSA/LSA1.kicad_pcb (KiCad board)
At the start: 2 copper layers, 61 x 33.1 mm, 20 parts, among them J1 Conn_02x05_Odd_Even, P1 D_Photo, P2 D_Photo, P3 D_Photo, P4 D_Photo, U1 LM324N_NOPB

Commit message: Updated resources
Routing:
- net GND: track 69.8 -> 180.1 mm
- net Net-(D3-Pad2): track 0.00 -> 2.62 mm
- net Net-(D2-Pad2): track 0.00 -> 2.35 mm
- net A1: track 50.1 -> 51.1 mm
